File: Schematic/Universal-Sensor_Atmega328.brd (EAGLE design)
At the start: 51.9 x 64.1 mm, 62 parts, among them IC1 Atmega 328P, IC2 MAX1724, IC3 TSL2561T, IC4 BMP180, IC5 SHT1X, IC6 MC34063-SO, IC7 AP7313-33SA, IC8 LT1785CS8, J3 I2C, Q1 CSTCXCSTCC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

Commit message: update board file
Routing:
- net GND: track 251.8 -> 252.0 mm, vias 126 -> 125
Other:
- board text added: "Rev 1.3, 11/2015"
- board text removed: "Rev 1.3, 07/2014"
